File: PowerSupply30V5A.kicad_sch (KiCad schematic)
At the start: 81 parts, among them IC4 MC7815BDTRKG, IC5 MC7812BDTRKG, IC6 MC7805BDTRKG, IC7 MC7915BD2TR4G, J1 1017503, J2 1017503, J3 76825-0004, J4 39300020, J5 76825-0004, J6 1017503, Q1 IRFP460, T1 AVB2.3_2_15, U1 ADA4062-2ARMZ, U2 ADA4062-2ARMZ, U3 ADA4062-2ARMZ

Commit message: Starting v2
Parts:
- added J7: ${FAMILY}, PHOENIX THD:PHOENIX_1755736, symbol Connectors:Connector 2 Male
- added TR1: 2x115V to 2x15V, Transformers:XFMR_BLOCK_FL14, symbol CERN_Windows:Transformers/XFMR_BLOCK_FL14/15
Other:
- note added: "1-Change components: Packaging, from Git library+ Standard components 1.1- Connectors need to select considering clearance-Creepage: I have six connectors * 220V AC INPUT- For 15/-15V trafo * 30V AC INPUT - From external trafo and directly to rectifier * Output of the PSU- +- Terminals (Can be +30V/5A) * Fan Supply OUTPUT- Try to test at 15V * V_ref-I_ref INPUT (With 5V OUTPUT) * V_out and I_out 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"
- note added: "How to calculate current? How to calculate power? The one I had before is 2.3 VA, the one of CernLib is 14VA. Need to calculate how much current I need and oversize x2 or similar, but no more. Secondary of the transformer is 30V, how many AMPS? For this I need to know how much they can my IC supply."
- moved on the sheet: BR1, BR2, C1, C10, C11, C12, C13, C14, C15, C16, C2, C3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

Commit message: Updates following steps
Parts:
- added BR3: MB1F, USER_BRIDGE_RECTIFIER:MB4F, symbol MB1F:MB1F
- added C17, C18: 1000uF, Capacitor_THT:C_Radial_D18.0mm_H35.5mm_P7.50mm, symbol Device:C_Polarized
- added C19, C20: 0.33uF, Capacitor_SMD:C_1206_3216Metric_Pad1.33x1.80mm_HandSolder, symbol Device:C
- added C21, C22: 0.1uF, Capacitor_SMD:C_0805_2012Metric_Pad1.18x1.45mm_HandSolder, symbol Device:C
- added IC1: MC7915BD2TR4G, USER_LDO:MC7915BD2TR4G, symbol MC7915BD2TR4G:MC7915BD2TR4G
- added IC2: MC7815BDTRKG, USER_LDO:NVD5117PLT4GVF01, symbol MC7815BDTRKG:MC7815BDTRKG
- added TP11, TP12: TestPoint, Connector_Pin:Pin_D0.7mm_L6.5mm_W1.8mm_FlatFork, symbol Connector:TestPoint
Connections:
- net +15V: now also C22.1, IC2.3 (OUT), TP12.1
- net -15V: now also C21.1, IC1.3 (OUT), TP11.1
- net GND: now also C17.2, C18.1, C19.2, C20.2, C21.2, C22.2, IC1.1 (GND), IC2.2 (GND)
- new net: C17.1, C20.1, IC2.1 (IN)
- new net: C18.2, C19.1, IC1.2 (IN)
Other:
- note added: "1-Change components: Packaging, from Git library+ Standard components+ IMPORTANT TO TRY TO REUSE IF IT WORKS what I already have 1.1- Connectors need to select considering clearance-Creepage: I have six connectors * 220V AC INPUT- For 15/-15V trafo * 30V AC INPUT - From external trafo and directly to rectifier * Output of the PSU- +- Terminals (Can be +30V/5A) * Fan Supply OUTPUT- Try to test at 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"
- note added: "All the components that I have here: I need to have them syncronised in the gitlab repository"
- note added: "Change for: PHOENIX 1939633"
- note added: "GO BACKWARDS: START FROM LDO's TO BRIDGE RECTIFIER CURRENT, AND THEN TRAFO POWER AND CONNECTOR"
- note added: "I_out(max)= 0.8A"
- note added: "Is it enough? Probably fan needs higher currents: Usually fans they are 12-24V: But what happens if I can supply it at 15V? I need to test it. Probably I need higher current and therefore a more powerfull trafo?"
- note removed: "1-Change components: Packaging, from Git library+ Standard components 1.1- Connectors need to select considering clearance-Creepage: I have six connectors * 220V AC INPUT- For 15/-15V trafo * 30V AC INPUT - From external trafo and directly to rectifier * Output of the PSU- +- Terminals (Can be +30V/5A) * Fan Supply OUTPUT- Try to test at 15V * V_ref-I_ref INPUT (With 5V OUTPUT) * V_out and I_out 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"

Commit message: Added LDO symbol with synch
Parts:
- removed IC2: MC7815BDTRKG, USER_LDO:NVD5117PLT4GVF01, symbol MC7815BDTRKG:MC7815BDTRKG
- added IC3: MC7815BDTRKG, m_LDO:NVD5117PLT4GVF01, symbol m_LDO:MC7815BDTRKG
Changed lines of the file:
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@@
 	)
 	(junction
-		(at 189.23 38.1)
-		(diameter 0)
-		(color 0 0 0 0)
-	)
-	(junction
 		(at 133.35 -115.57)
 		(diameter 0)
@@
 	)
 	(symbol
+		(lib_id "m_LDO:MC7815BDTRKG")
+		(at 104.14 82.55 0)
+		(unit 1)
+		(exclude_from_sim no)
+		(in_bom yes)
+		(on_board yes)
+		(dnp no)
+		(property "Reference" "IC3"
+			(at 125.73 74.93 0)
+			(effects
+				(font
+					(size 1.27 1.27)
+				)
+				(justify left top)
+			)
+		)
+		(property "Value" "MC7815BDTRKG"
+			(at 125.73 77.47 0)
+			(effects
+				(font
+					(size 1.27 1.27)
+				)
+				(justify left top)
+			)
+		)
+		(property "Footprint" "m_LDO:NVD5117PLT4GVF01"
+			(at 125.73 177.47 0)
+			(effects
+				(font
+					(size 1.27 1.27)
+				)
+				(justify left top)
+				(hide yes)
+			)
+		)
+		(property "Datasheet" "https://www.onsemi.com/pub/Collateral/MC7800-D.PDF"
+			(at 125.73 277.47 0)
+			(effects
+				(font
+					(size 1.27 1.27)
+				)
+				(justify left top)
+				(hide yes)
+			)
+		)
+		(property "Description" "Output Current in Excess of 1.0 A; No External Components Required; Internal Thermal Overload Protection; Internal Short Circuit Current Limiting; Output Transistor Safe-Area Compensation; Output Voltage Offered in 2% and 4% Tolerance; Pb-Free Packages are Available"
+			(at 104.14 82.55 0)
+			(effects
+				(font
+					(size 1.27 1.27)
+				)
+				(hide yes)
+			)
+		)
+		(property "Height" "2.38"
+			(at 125.73 477.47 0)
+			(effects
+				(font
+					(size 1.27 1.27)
+				)
+				(justify left top)
+				(hide yes)
+			)
+		)
+		(property "Manufacturer_Name" "onsemi"
+			(at 125.73 577.47 0)
+			(effects
+				(font
+					(size 1.27 1.27)
+				)
+				(justify left top)
+				(hide yes)
+			)
+		)
+		(property "Manufacturer_Part_Number" "MC7815BDTRKG"
+			(at 125.73 677.47 0)
+			(effects
+				(font
+					(size 1.27 1.27)
+				)
+				(justify left top)
+				(hide yes)
+			)
+		)
+		(property "Mouser Part Number" "863-MC7815BDTRKG"
+			(at 125.73 777.47 0)
+			(effects
+				(font
+					(size 1.27 1.27)
+				)
+				(justify left top)
+				(hide yes)
+			)
+		)
+		(property "Mouser Price/Stock" "https://www.mouser.co.uk/ProductDetail/onsemi/MC7815BDTRKG?qs=%252B9%2Fcbd0IE0QAayqLvnGs6g%3D%3D"
+			(at 125.73 877.47 0)
+			(effects
+				(font
+					(size 1.27 1.27)
+				)
+				(justify left top)
+				(hide yes)
+			)
+		)
+		(property "Arrow Part Number" "MC7815BDTRKG"
+			(at 125.73 977.47 0)
+			(effects
+				(font
+					(size 1.27 1.27)
+				)
+				(justify left top)
+				(hide yes)
+			)
+		)
+		(property "Arrow Price/Stock" "https://www.arrow.com/en/products/mc7815bdtrkg/on-semiconductor?region=nac"
+			(at 125.73 1077.47 0)
+			(effects
+				(font
+					(size 1.27 1.27)
+				)
+				(justify left top)
+				(hide yes)
+			)
+		)
+		(pin "2"
+		)
+		(pin "3"
+		)
+		(pin "1"
+		)
+		(instances
+			(project ""
+				(path "/47083ad7-9fa0-4f9a-906f-7d13aa6ff8f4"
+					(reference "IC3")
+					(unit 1)
+				)
+			)
+		)
+	)
+	(symbol
 		(lib_id "76825-0004:76825-0004")
 		(at 71.12 -26.67 0)
@@
 					(unit 1)
 				)
-			)
-		)
-	)
-	(symbol
-		(lib_id "MC7815BDTRKG:MC7815BDTRKG")
-		(at 163.83 38.1 0)
-		(unit 1)
-		(exclude_from_sim no)
-		(in_bom yes)
-		(on_board yes)
-		(dnp no)
-		(fields_autoplaced yes)
-		(property "Reference" "IC2"
-			(at 176.53 30.48 0)
-			(effects
-				(font
-					(size 1.27 1.27)
-				)
-			)
-		)
-		(property "Value" "MC7815BDTRKG"
-			(at 176.53 33.02 0)
-			(effects
-				(font
-					(size 1.27 1.27)
-				)
-			)
-		)
-		(property "Footprint" "USER_LDO:NVD5117PLT4GVF01"
-			(at 185.42 133.02 0)
-			(effects
-				(font
-					(size 1.27 1.27)
-				)
-				(justify left top)
-				(hide yes)
-			)
-		)
-		(property "Datasheet" "https://www.onsemi.com/pub/Collateral/MC7800-D.PDF"
-			(at 185.42 233.02 0)
-			(effects
-				(font
-					(size 1.27 1.27)
-				)
-				(justify left top)
-				(hide yes)
-			)
-		)
-		(property "Description" "Output Current in Excess of 1.0 A; No External Components Required; Internal Thermal Overload Protection; Internal Short Circuit Current Limiting; Output Transistor Safe-Area Compensation; Output Voltage Offered in 2% and 4% Tolerance; Pb-Free Packages are Available"
-			(at 163.83 38.1 0)
-			(effects
-				(font
-					(size 1.27 1.27)
-				)
-				(hide yes)
-			)
-		)
-		(property "Height" "2.38"
-			(at 185.42 433.02 0)
-			(effects
-				(font
-					(size 1.27 1.27)
-				)
-				(justify left top)
-				(hide yes)
-			)
-		)
-		(property "Manufacturer_Name" "onsemi"
-			(at 185.42 533.02 0)
-			(effects
-				(font
-					(size 1.27 1.27)
-				)
-				(justify left top)
-				(hide yes)
-			)
-		)
-		(property "Manufacturer_Part_Number" "MC7815BDTRKG"
-			(at 185.42 633.02 0)
-			(effects
-				(font
-					(size 1.27 1.27)
-				)
-				(justify left top)
-				(hide yes)
-			)
-		)
-		(property "Mouser Part Number" "863-MC7815BDTRKG"
-			(at 185.42 733.02 0)
-			(effects
-				(font
-					(size 1.27 1.27)
-				)
-				(justify left top)
-				(hide yes)
-			)
-		)
-		(property "Mouser Price/Stock" "https://www.mouser.co.uk/ProductDetail/onsemi/MC7815BDTRKG?qs=%252B9%2Fcbd0IE0QAayqLvnGs6g%3D%3D"
-			(at 185.42 833.02 0)
-			(effects
-				(font
-					(size 1.27 1.27)
-				)
-				(justify left top)
-				(hide yes)
-			)
-		)
-		(property "Arrow Part Number" "MC7815BDTRKG"
-			(at 185.42 933.02 0)
-			(effects
-				(font
-					(size 1.27 1.27)
-				)
-				(justify left top)
-				(hide yes)
-			)
-		)
-		(property "Arrow Price/Stock" "https://www.arrow.com/en/products/mc7815bdtrkg/on-semiconductor?region=nac"
-			(at 185.42 1033.02 0)
-			(effects
-				(font
-					(size 1.27 1.27)
-				)
-				(justify left top)
-				(hide yes)
-			)
-		)
-		(pin "1"
-		)
-		(pin "3"
-		)
-		(pin "2"
-		)
-		(instances
-			(project "PowerSupply30V5A"
-				(path "/47083ad7-9fa0-4f9a-906f-7d13aa6ff8f4"
-					(reference "IC2")
-					(unit 1)
-				)

Commit message: Added -15V LDO
Parts:
- removed IC1: MC7915BD2TR4G, USER_LDO:MC7915BD2TR4G, symbol MC7915BD2TR4G:MC7915BD2TR4G
- removed IC3: MC7815BDTRKG, m_LDO:NVD5117PLT4GVF01, symbol m_LDO:MC7815BDTRKG
- added IC2: MC7815BDTRKG, m_LDO:NVD5117PLT4GVF01, symbol m_LDO:MC7815BDTRKG
- added IC3: MC7915BD2TR4G, m_LDO:MC7915BD2TR4G, symbol m_LDO:MC7915BD2TR4G
- C21: value 0.1uF -> 1uF
- C22: value 0.1uF -> 1uF; footprint Capacitor_SMD:C_0805_2012Metric_Pad1.18x1.45mm_HandSolder -> Capacitor_SMD:C_1206_3216Metric_Pad1.33x1.80mm_HandSolder
Connections:
- net +15V: now also IC2.3 (OUT)
- net -15V: now also IC3.3 (OUT)
- net GND: now also IC2.2 (GND), IC3.1 (GND)
- net at C17.1, C20.1: now also IC2.1 (IN)
- net at C18.2, C19.1: now also IC3.2 (IN)
Other:
- note added: "C_out lower than 0.1uF causes instabilities"
- note added: "I believe this was not working properly cause I was asking more current than possible"
- note added: "I_out(max): 1A (With heatsink)"
- note added: "LDO Dropout voltage: 2V So for 15V I need 18Vmin in the output"
- note added: "LDO dropout voltage: 1.3V So for -15v I need -18.7Vmin"
- note added: "NEXT: Do the same with 12V (if needed) and 5V ldo, and once done, size correctly this time trafo, rectifier and connector"
- note added: "Should I choose D2PAK for both? or try to reuse what I already have"
- note added: "This might be needed to be +-18V trafo, and more powerfull (that is why I was not having enough)"

Commit message: Added additional todo
Other:
- note added: "Need to understand when is stored kicad_symbol, cause I cannot see it in the kicad.sym folder: What happens if I try to open somewhere else?"
Changed lines of the file:
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@@
+		)
+	)
+	(text "Need to understand when is stored kicad_symbol, cause I cannot see it in the kicad.sym folder: What happens if I try to open somewhere else? "
+		(exclude_from_sim no)
+		(at -78.994 33.782 0)
+		(effects
+			(font
+				(size 1.27 1.27)
+			)
 		)
 	)

Commit message: Added 5V and 12 V LDO, started with mosfet side, corrected 50mOhm resistor
Parts:
- added BR4: KBJB1506_T0_00301, USER_BRIDGE_RECTIFIER_2:KBJB1506_T0_00301, symbol KBJB1506_T0_00301:KBJB1506_T0_00301
- added C23, C25: 0.33uF, Capacitor_SMD:C_1206_3216Metric_Pad1.33x1.80mm_HandSolder, symbol Device:C
- added C24, C26: 1uF, Capacitor_SMD:C_1206_3216Metric_Pad1.33x1.80mm_HandSolder, symbol Device:C
- added C27, C28, C29: 1000uF, Capacitor_THT:C_Radial_D18.0mm_H35.5mm_P7.50mm, symbol Device:C_Polarized
- added IC1: MC7805BDTRKG, m_LDO:LM317MADTRKG, symbol m_LDO:MC7805BDTRKG
- added IC9: MC7812BDTRKG, m_LDO:MC7812BDTRKG, symbol m_LDO:MC7812BDTRKG
- added J8, J9: 1017503, USER_CONNECTOR_2:CONN_1017491, symbol 2026-01-31_20-20-20:1017503
- added Q2: IRFP460, USER_MOSFET:TO546P1587X531X2511-3, symbol IRFP460:IRFP460
- added R28: 10kΩ, Resistor_SMD:R_2512_6332Metric_Pad1.40x3.35mm_HandSolder, symbol Device:R
- added R30: Y14870R05000B9R, m_Resistor_measurement:Y14870R05000B9R, symbol m_Resistor_measurement:Y14870R05000B9R
- added TP13, TP14: TestPoint, Connector_Pin:Pin_D0.7mm_L6.5mm_W1.8mm_FlatFork, symbol Connector:TestPoint
Connections:
- net +12V: now also C23.1, C26.1, IC1.1 (IN), IC9.3 (OUT), TP14.1
- net +15V: now also C25.1, IC9.1 (IN)
- net +5V: now also C24.1, IC1.3 (OUT), TP13.1
- net 0V_IN: now also BR4.4 (-), C27.2, C28.2, C29.2, J9.3, J9.4
- net 30V_IN: now also BR4.1 (+), C27.1, C29.1, Q2.2
- net GND: now also C23.2, C24.2, C25.2, C26.2, IC1.2 (GND), IC9.2 (GND), Q2.3
- net I_OUT_MEAS-: now also C28.1, J9.1, J9.2
- net V_GATE: now also R28.1
- new net: Q2.1, R28.2
- new net: BR4.2 (~_1), J8.3, J8.4
- new net: BR4.3 (~_2), J8.1, J8.2
Other:
- note added: "Did I actually order 1mOhm resistor instead of 50mOhm? Yes: change for: Y14870R05000B9R"
- note added: "LDO dropout voltage: 2V So for 12v I need 14.5Vmin"
- note added: "LDO dropout voltage: 2V So for 5v I need 7.5Vmin"
- note added: "NEXT: Do the same with 12V (if needed- Can i use another fan?) and 5V ldo, and once done, size correctly this time trafo, rectifier and connector"
- note added: "Need to calculate current needed to be delivered by these LDO"
- note added: "P_max=5W 05"
- note added: "Should I choose D2PAK for both? or try to reuse what I already have. If I have extra, I can reuse: Otherwise, I can use same packaging for all of them"
- note added: "To be finished later"
- note removed: "NEXT: Do the same with 12V (if needed) and 5V ldo, and once done, size correctly this time trafo, rectifier and connector"
- note removed: "Should I choose D2PAK for both? or try to reuse what I already have"
- moved on the sheet: C18, C19, C21, IC3, TP11

Commit message: Advanced in power mosfet stage
Parts:
- removed J9: 1017503, USER_CONNECTOR_2:CONN_1017491, symbol 2026-01-31_20-20-20:1017503
- removed Q2: IRFP460, USER_MOSFET:TO546P1587X531X2511-3, symbol IRFP460:IRFP460
- removed R30: Y14870R05000B9R, m_Resistor_measurement:Y14870R05000B9R, symbol m_Resistor_measurement:Y14870R05000B9R
- added J11: 1017503, m_Connectors:1017503, symbol m_Connectors:1017503
- added Q3: IRFP460, m_MOSFET:TO546P1587X531X2511-3, symbol m_MOSFET:IRFP460
- added R29: Y14870R05000B9R, m_Resistor_measurement:Y14870R05000B9R, symbol m_Resistor_measurement:Y14870R05000B9R
- added R30: FCSL76R050DER, m_Resistor_measurement:RESC3876X70N, symbol m_Resistor_measurement:FCSL76R050DER
Connections:
- net 0V_IN: now also J11.3, J11.4
- net 30V_IN: now also Q3.2
- net GND: now also Q3.3
- net I_OUT_MEAS-: now also J11.1, J11.2
- net at R28.2: now also Q3.1
Other:
- note added: "Choose one brand for resistors and capacitors, SMD, 1206, so that I can order a huge catalogue: chrome-extension://efaidnbmnnnibpcajpcglclefindmkaj/https://www.vishay.com/docs/20132/rca-sre3.pdf"
- note added: "NEXT: Power MOSFET stage"
- note added: "P_max_operation=1.25W(50mOhms*(5A)^2)"
- note removed: "NEXT: Do the same with 12V (if needed- Can i use another fan?) and 5V ldo, and once done, size correctly this time trafo, rectifier and connector"
- note removed: "P_max=5W 05"
- moved on the sheet: C28

Commit message: Continued with Power MOSFET STAGE
Parts:
- removed C29: 1000uF, Capacitor_THT:C_Radial_D18.0mm_H35.5mm_P7.50mm, symbol Device:C_Polarized
- removed J8: 1017503, USER_CONNECTOR_2:CONN_1017491, symbol 2026-01-31_20-20-20:1017503
- removed R28: 10kΩ, Resistor_SMD:R_2512_6332Metric_Pad1.40x3.35mm_HandSolder, symbol Device:R
- removed R29: Y14870R05000B9R, m_Resistor_measurement:Y14870R05000B9R, symbol m_Resistor_measurement:Y14870R05000B9R
- added J8: ${FAMILY}, PHOENIX THD:PHOENIX_1755736, symbol Connectors:Connector 2 Male
- added R28: 10kΩ, m_Resistor_SMD:RESC3216X60N, symbol m_Resistor_SMD:RCA120610K0JNEASR
Connections:
- net GND: now also R30.1
- net I_OUT_MEAS-: now also R30.2
- net V_GATE: now also R28. (2)
- net at Q3.1: now also R28. (2)
- net at BR4.2 (~_1): now also J8.1
- net at BR4.3 (~_2): now also J8.2
Other:
- note added: "For current measurement: Did I actually order 1mOhm resistor instead of 50mOhm?"
- note added: "NEXT: Power MOSFET stage-Missing calculation for rectifier: Not done for any of them"
- note added: "THINGS I WAS DOING WRONG IN V1:"
- note added: "Why I don´t use same power rectifier? One has +-15Vac(So 30V)- But is true it has less current The other one is also +30Vac, but requires much more power. Need to calculate this"
- note removed: "Did I actually order 1mOhm resistor instead of 50mOhm? Yes: change for: Y14870R05000B9R"
- note removed: "NEXT: Power MOSFET stage"
- moved on the sheet: C27, C28, J11
