File: PowerSupply30V5A.kicad_sch (KiCad schematic)
At the start: 157 parts, among them IC1 MC7805BDTRKG, IC10 LF247DT, IC2 MC7815BDTRKG, IC3 MC7915BD2TR4G, IC4 MC7815BDTRKG, IC5 MC7812BDTRKG, IC6 MC7805BDTRKG, IC7 MC7915BD2TR4G, IC8 LF247DT, IC9 MC7812BDTRKG, J1 1017503, J10 1755752, J11 1017503, J12 ${FAMILY}, J2 1017503, J3 76825-0004, J4 39300020, J5 76825-0004, J6 1017503, J7 ${FAMILY}, J8 ${FAMILY}, J9 1755752, Q1 IRFP460, Q3 IRFP460, T1 AVB2.3_2_15, U1 ADA4062-2ARMZ, U2 ADA4062-2ARMZ, U3 ADA4062-2ARMZ

Commit message: Substituted all the capas for my library
Parts:
- removed C19, C20, C23, C25: 0.33uF, Capacitor_SMD:C_1206_3216Metric_Pad1.33x1.80mm_HandSolder, symbol Device:C
- removed C29, C32, C34, C36: 0.1uF, Capacitor_SMD:C_1206_3216Metric_Pad1.33x1.80mm_HandSolder, symbol Device:C
- removed C33, C35: 4.7nF, Capacitor_SMD:C_1206_3216Metric_Pad1.33x1.80mm_HandSolder, symbol Device:C
- added C19, C20, C23, C26: 330nF_25V, m_Capacitor_ceramic_SMD:CAPC2012X94N, symbol m_Capacitor_ceramic_SMD:0805_330nF_25V_10%
- added C25, C29, C32, C34: 100nF_50V, m_Capacitor_ceramic_SMD:CAPC2012X94N, symbol m_Capacitor_ceramic_SMD:0805_100nF_50V_10%
- added C33, C36: 4.7nF_50V, m_Capacitor_ceramic_SMD:CAPC2012X94N, symbol m_Capacitor_ceramic_SMD:0805_4.7nF_50V_5%
Connections:
- net +12V: now also C26. (2)
- net +15V: now also C23. (2), C25. (2)
- net -15V: now also C29. (2)
- net 0V_IN: now also C32. (2)
- net GND: now also C19. (2), C20. (2), C23. (2), C25. (2), C26. (2), C29. (2)
- net I_control: now also C33. (2)
- net V_MEAS: now also C34. (2)
- net V_control: now also C36. (2)
- net at R37. (2): now also IC8.2 (-), R36. (2); no longer R38. (2)
- net at R49. (2): now also IC8.6 (-), R48. (2); no longer R50. (2)
- net at C17.1, IC2.1 (IN): now also C20. (2)
- net at C18.2, IC3.2 (IN): now also C19. (2)
- new net: R37. (2), R38. (2)
- new net: R49. (2), R50. (2)
- new net: C36. (2), IC8.13 (-), R55. (2), R56. (2)
- new net: IC8.10 (+), R39. (2), R40. (2)
- new net: C34. (2), IC8.12 (+), R53. (2), R54. (2)
- new net: IC8.3 (+), R30. (2), R44. (2)
- new net: C32. (2), IC8.5 (+), R47. (2), R51. (2)
- new net: C33. (2), IC8.9 (-), R41. (2), R42. (2)

Commit message: Calculated power comsumption by +5V and +12V rails
Connections:
- net at R37. (2): now also IC8.2 (-), R36. (2); no longer R38. (2)
- net at R49. (2): now also IC8.6 (-), R48. (2); no longer R50. (2)
- new net: R37. (2), R38. (2)
- new net: R49. (2), R50. (2)
- new net: C36. (2), IC8.13 (-), R55. (2), R56. (2)
- new net: IC8.10 (+), R39. (2), R40. (2)
- new net: C34. (2), IC8.12 (+), R53. (2), R54. (2)
- new net: IC8.3 (+), R30. (2), R44. (2)
- new net: C32. (2), IC8.5 (+), R47. (2), R51. (2)
- new net: C33. (2), IC8.9 (-), R41. (2), R42. (2)
Other:
- note added: "* Fan: Need to calculate @home. For the moment lets say 1A * Voltage presence indicator: 20mA * Mosfet Gate driver: Imax-=0.5A > When MOSFET fully closed (Current dissipated in 20Ω): 6V/20Ω=0.3A > When MOSFET fully opened (Current dissipated in 10Ω+ Diode voltage drop): (6V-1V)/10Ω=0.5A * LDO 5V: P_LDO= (V_in-V_out)*I_out + V_in*Iq (Quiescent current)= 2V*1A+12V*3.2mA= 2.0384W * P_tot_12V= [12V *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"
- note added: "* Voltage presence indicator: 20mA * For current and voltage reference: 1.25W > Scenario with potentiometer: Need to measure: For the moment I remember 50mOhm = 5V^2/50mOhm=1.25W > Scenario with MCU: I will not need this reference, voltage will be given by MCU. * P_tot_5V= (5V*20e-3)+1.25W= 1.35W"
- note added: "+12V: (20.27W)"
- note added: "+15V: (xx W)"
- note added: "+5V: (1.35W)"
- note added: "-15V: (xx W)"
- note added: "I_out(max): 1A (With heatsink) P_out= 5V*1A=5W"
- note added: "NEXT(X2): Electrical check +testpoints"
- note added: "Power of the board for each voltage rail (and LDO):"
- note removed: "All capacitors library are missing: I need to replace both electrolitic and ceramic ones"
- note removed: "Choose one brand for resistors and capacitors, SMD, 1206, so that I can order a huge catalogue: chrome-extension://efaidnbmnnnibpcajpcglclefindmkaj/https://www.vishay.com/docs/20132/rca-sre3.pdf"
- note removed: "NEXT(X2): Capacitor library+ Electrical check +testpoints"
- note removed: "NEXT: 1uF changed , add other values by copy pasting Capacitor select 1206 (Correccion, no tiene sentido que todos sean iguales) Lo que puedo encontrar es un kit ya preparado (Y comprar una vez:) Luego contemplar si deberia de hacer lo mismo con las resistencias https://www.mouser.co.uk/en/ProductDetail/Wurth-Elektronik/885070?qs=%252BUQ4csG8RsciqaV%252BTbV4fQ%3D%3D"
Changed lines of the file:
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@@
 	(rectangle
 		(start -132.08 35.56)
-		(end -62.23 44.45)
+		(end -62.23 46.99)
 		(stroke
 			(width 0)
@@
 		)
 	)
-	(text "NEXT:  1uF changed , add other values by copy pasting\nCapacitor select 1206 (Correccion, no tiene sentido que todos sean iguales)\nLo que puedo encontrar es un kit ya preparado (Y comprar una vez:)\nLuego contemplar si deberia de hacer lo mismo con las resistencias\nhttps://www.mouser.co.uk/en/ProductDetail/Wurth-Elektronik/885070?qs=%252BUQ4csG8RsciqaV%252BTbV4fQ%3D%3D"
-		(exclude_from_sim no)
-		(at -101.346 28.194 0)
-		(effects
-			(font
-				(size 1.27 1.27)
-				(color 51 255 30 1)
-			)
-		)
-	)
 	(text "Voltage sensing"
 		(exclude_from_sim no)
@@
 		)
 	)
+	(text "Power of the board for each voltage rail (and LDO):"
+		(exclude_from_sim no)
+		(at 458.724 38.608 0)
+		(effects
+			(font
+				(size 1.27 1.27)
+				(thickness 0.254)
+				(bold yes)
+			)
+		)
+	)
 	(text "POWER CONTROL\n"
 		(exclude_from_sim no)
@@
 		)
 	)
-	(text "I_out(max): 1A (With heatsink)"
-		(exclude_from_sim no)
-		(at 258.318 93.98 0)
+	(text "I_out(max): 1A (With heatsink)\nP_out= 5V*1A=5W\n\n"
+		(exclude_from_sim no)
+		(at 258.318 92.71 0)
 		(effects
 			(font
@@
 			(font
 				(size 1.27 1.27)
+			)
+		)
+	)
+	(text "+15V: (xx W)"
+		(exclude_from_sim no)
+		(at 441.96 77.724 0)
+		(effects
+			(font
+				(size 1.27 1.27)
+				(thickness 0.254)
+				(bold yes)
 			)
 		)
@@
 		)
 	)
-	(text "NEXT(X2): Capacitor library+ Electrical check +testpoints"
+	(text "* Voltage presence indicator: 20mA\n* For current and voltage reference: 1.25W\n 	> Scenario with potentiometer: Need to measure: For the moment I remember 50mOhm = 5V^2/50mOhm=1.25W\n	> Scenario with MCU: I will not need this reference, voltage will be given by MCU. \n* P_tot_5V= (5V*20e-3)+1.25W= 1.35W"
+		(exclude_from_sim no)
+		(at 436.118 69.342 0)
+		(effects
+			(font
+				(size 1.27 1.27)
+			)
+			(justify left)
+		)
+	)
+	(text "NEXT(X2): Electrical check +testpoints"
 		(exclude_from_sim no)
 		(at -101.092 42.926 0)
@@
 		)
 	)
+	(text "+12V: (20.27W)"
+		(exclude_from_sim no)
+		(at 440.944 42.164 0)
+		(effects
+			(font
+				(size 1.27 1.27)
+				(thickness 0.254)
+				(bold yes)
+			)
+		)
+	)
 	(text "LDO dropout voltage: 2V\nSo for 5v I need 7.5Vmin"
 		(exclude_from_sim no)
-		(at 257.556 90.678 0)
+		(at 257.556 87.122 0)
 		(effects
 			(font
@@
 	(text "Una vez terminado: Hacer check electrico del esquematico+ actualizar numeros"
 		(exclude_from_sim no)
-		(at -103.378 58.166 0)
+		(at -100.076 48.768 0)
 		(effects
 			(font
@@
 			(font
 				(size 1.27 1.27)
-			)
-		)
-	)
-	(text "Choose one brand for resistors and capacitors, SMD, 1206, so that I can order a huge catalogue:\nchrome-extension://efaidnbmnnnibpcajpcglclefindmkaj/https://www.vishay.com/docs/20132/rca-sre3.pdf"
-		(exclude_from_sim no)
-		(at -93.218 70.866 0)
-		(effects
-			(font
-				(size 1.27 1.27)
-				(color 25 255 113 1)
 			)
 		)
@@
 		)
 	)
-	(text "All capacitors library are missing: I need to replace both electrolitic and ceramic ones\n"
-		(exclude_from_sim no)
-		(at -100.076 47.498 0)
-		(effects
-			(font
-				(size 1.27 1.27)
-				(color 255 12 12 1)
-			)
-		)
-	)
 	(text "THINGS I WAS DOING WRONG IN V1:"
 		(exclude_from_sim no)
@@
 		)
 	)
-	(text "change opamp by proper opamp schematic\n"
-		(exclude_from_sim no)
-		(at -101.854 335.28 0)
-		(effects
-			(font
-				(size 1.27 1.27)
-			)
-		)
-	)
-	(text "VOLTAGE PRESENCE INDICATOR\n"
-		(exclude_from_sim no)
-		(at 332.74 33.02 0)
+	(text "-15V: (xx W)"
+		(exclude_from_sim no)
+		(at 441.96 84.836 0)
 		(effects
 			(font
@@
 		)
 	)
+	(text "change opamp by proper opamp schematic\n"
+		(exclude_from_sim no)
+		(at -101.854 335.28 0)
+		(effects
+			(font
+				(size 1.27 1.27)
+			)
+		)
+	)
+	(text "VOLTAGE PRESENCE INDICATOR\n"
+		(exclude_from_sim no)
+		(at 332.74 33.02 0)
+		(effects
+			(font
+				(size 1.27 1.27)
+				(thickness 0.254)
+				(bold yes)
+			)
+		)
+	)
 	(text "After simply design this one\n"
 		(exclude_from_sim no)
@@
 		)
 	)
+	(text "* Fan: Need to calculate @home. For the moment lets say 1A\n* Voltage presence indicator: 20mA\n* Mosfet Gate driver: Imax-=0.5A\n	> When MOSFET fully closed (Current dissipated in 20Ω): 6V/20Ω=0.3A\n	> When MOSFET fully opened (Current dissipated in 10Ω+ Diode voltage drop): (6V-1V)/10Ω=0.5A\n* LDO 5V: P_LDO= (V_in-V_out)*I_out + V_in*Iq (Quiescent current)= 2V*1A+12V*3.2mA= 2.0384W\n* P_tot_12V= [12V * (1+20e-3+0.5)]+2.0384=20.27W"
+		(exclude_from_sim no)
+		(at 435.61 51.308 0)
+		(effects
+			(font
+				(size 1.27 1.27)
+				(thickness 0.1588)
+			)
+			(justify left)
+		)
+	)
 	(text "FAN+"
 		(exclude_from_sim no)
@@
 				(size 1.27 1.27)
 				(color 255 5 20 1)
+			)
+		)
+	)
+	(text "+5V: (1.35W)"
+		(exclude_from_sim no)
+		(at 440.944 62.23 0)
+		(effects
+			(font
+				(size 1.27 1.27)
+				(thickness 0.254)
+				(bold yes)
 			)
 		)
@@
 		)
 	)
-	(polyline
-		(pts
-			(xy 36.83 213.36) (xy 114.3 213.36)
-		)
-		(stroke
-			(width 0)
-			(type dash)
-		)
-	)

Commit message: Missing current measurement of the fan to finish calculating power
Parts:
- added C35: 100nF_50V, m_Capacitor_ceramic_SMD:CAPC2012X94N, symbol m_Capacitor_ceramic_SMD:0805_100nF_50V_10%
- added C38: 1μF_25V, m_Capacitor_ceramic_SMD:CAPC2012X94N, symbol m_Capacitor_ceramic_SMD:0805_1μF_25V_20%
Connections:
- net +15V: now also C35. (2), C38. (2)
- net GND: now also C35. (2), C38. (2)
- net at R37. (2): now also IC8.2 (-), R36. (2); no longer R38. (2)
- net at R49. (2): now also IC8.6 (-), R48. (2); no longer R50. (2)
- new net: R37. (2), R38. (2)
- new net: R49. (2), R50. (2)
- new net: C36. (2), IC8.13 (-), R55. (2), R56. (2)
- new net: IC8.10 (+), R39. (2), R40. (2)
- new net: C34. (2), IC8.12 (+), R53. (2), R54. (2)
- new net: IC8.3 (+), R30. (2), R44. (2)
- new net: C32. (2), IC8.5 (+), R47. (2), R51. (2)
- new net: C33. (2), IC8.9 (-), R41. (2), R42. (2)
Other:
- note added: "* Fan: Need to calculate @home. For the moment lets say 1A * Voltage presence indicator: 20mA * Mosfet Gate driver: Imax-=0.5A > When MOSFET fully closed (Current dissipated in 20Ω): 6V/20Ω=0.3A > When MOSFET fully opened (Current dissipated in 10Ω+ Diode voltage drop): (6V-1V)/10Ω=0.5A * LDO 5V: P_int_LDO_5V+ P_out_5V= (V_in-V_out)*I_out + V_in*Iq (Quiescent current)= 7*1A+12V*3.2mA= 7.0384W+1.3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"
- note added: "* Voltage presence indicator: 20mA * For current and voltage reference: 1.25W > Scenario with potentiometer: Need to measure: For the moment I remember 50mOhm = 5V^2/50mOhm=1.25W > Scenario with MCU: I will not need this reference, voltage will be given by MCU. * P_out_5V= (5V*20e-3)+1.25W= 1.35W"
- note added: "* Voltage presence indicator: 20mA * Quad op-amp buffer: 680mW Pmax when output @+15V * Quad op-amp voltage and current PI:680mW Pmax when output @+15V * LDO 12V: P_int_LDO_12V+P_out_12V= (V_in-V_out)*I_out + V_in*Iq (Quiescent current)= 3V*1A+18V*3.5mA= 3.063W * P_tot_15V"
- note added: "* Voltage presence indicator: 20mA * Quad op-amp buffer: 680mW Pmax when output @-15V * Quad op-amp voltage and current PI:680mW Pmax when output @-15V * P_tot_15V= (15V*20mA) + (2*680mW) = 1.66W"
- note added: "Claro, el opamp es 1A solo, asique tengo que medir esto. Si es 1A, tengo que cambiar LDO Aqui estoy dando 2A en el op-amp! no funciona"
- note added: "I_out_-15V=111mA"
- note added: "I_out_12V=2A"
- note added: "I_out_15V=xxA"
- note added: "I_out_5V=330mA"
- note added: "Y aqui cambiar P_out_12V una vez haya medido"
- note removed: "* Fan: Need to calculate @home. For the moment lets say 1A * Voltage presence indicator: 20mA * Mosfet Gate driver: Imax-=0.5A > When MOSFET fully closed (Current dissipated in 20Ω): 6V/20Ω=0.3A > When MOSFET fully opened (Current dissipated in 10Ω+ Diode voltage drop): (6V-1V)/10Ω=0.5A * LDO 5V: P_LDO= (V_in-V_out)*I_out + V_in*Iq (Quiescent current)= 2V*1A+12V*3.2mA= 2.0384W * P_tot_12V= [12V *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"
- note removed: "* Voltage presence indicator: 20mA * For current and voltage reference: 1.25W > Scenario with potentiometer: Need to measure: For the moment I remember 50mOhm = 5V^2/50mOhm=1.25W > Scenario with MCU: I will not need this reference, voltage will be given by MCU. * P_tot_5V= (5V*20e-3)+1.25W= 1.35W"

Commit message: update title
Parts:
- removed BR4: KBJB1506_T0_00301, USER_BRIDGE_RECTIFIER_2:KBJB1506_T0_00301, symbol KBJB1506_T0_00301:KBJB1506_T0_00301
- added BR5: KBJB1506_T0_00301, m_BridgeRectifier:KBJB1506_T0_00301, symbol m_BridgeRectifier:KBJB1506_T0_00301
Connections:
- net 0V_IN: now also BR5.4 (-)
- net 30V_IN: now also BR5.1 (+)
- net at R37. (2): now also IC8.2 (-), R36. (2); no longer R38. (2)
- net at R49. (2): now also IC8.6 (-), R48. (2); no longer R50. (2)
- net at J8.1: now also BR5.3 (~_2)
- net at J8.2: now also BR5.2 (~_1)
- new net: R37. (2), R38. (2)
- new net: R49. (2), R50. (2)
- new net: C36. (2), IC8.13 (-), R55. (2), R56. (2)
- new net: IC8.10 (+), R39. (2), R40. (2)
- new net: C34. (2), IC8.12 (+), R53. (2), R54. (2)
- new net: IC8.3 (+), R30. (2), R44. (2)
- new net: C32. (2), IC8.5 (+), R47. (2), R51. (2)
- new net: C33. (2), IC8.9 (-), R41. (2), R42. (2)
Other:
- note added: "+30V*5A=150W"
- note added: "Dont connect without heatsink"
- note added: "How can I know which is the voltage in the output, knowing the AC voltage?"
- note added: "NEXT: +Finish calculating current/power of LDO +Choose bridge rectifier+ transformer following from this"
- note added: "P_out=150W With heat sink:15A WIthout heatsin:3.2A!!"
- note added: "Power of the PSU rail:"
- note added: "Regulable Lab Power Supply Unit (PSU): 30V/5A"
- note added: "Write down properties of the trnasformer here"
Changed lines of the file:
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@@
 	)
 	(rectangle
+		(start 159.004 -2.54)
+		(end 258.064 5.08)
+		(stroke
+			(width 0)
+			(type default)
+		)
+		(fill
+			(type none)
+		)
+	)
+	(rectangle
 		(start 167.64 171.45)
 		(end 193.04 198.12)
@@
 	)
 	(rectangle
-		(start 63.5 60.96)
-		(end 87.63 83.82)
-		(stroke
-			(width 0)
-			(type solid)
-			(color 255 20 21 1)
-		)
-		(fill
-			(type none)
-		)
-	)
-	(rectangle
 		(start 22.86 147.32)
 		(end 123.19 267.97)
@@
 		)
 	)
+	(text "Dont connect without heatsink"
+		(exclude_from_sim no)
+		(at 99.568 73.66 0)
+		(effects
+			(font
+				(size 1.27 1.27)
+				(color 255 43 2 1)
+			)
+		)
+	)
 	(text "Voltage sensing"
 		(exclude_from_sim no)
@@
 		)
 	)
+	(text "How can I know which is the voltage in the output, \nknowing the AC voltage?"
+		(exclude_from_sim no)
+		(at 114.3 79.756 0)
+		(effects
+			(font
+				(size 1.27 1.27)
+				(color 255 45 39 1)
+			)
+		)
+	)
 	(text "30 AC- From \nHigh Power\nTransformer"
 		(exclude_from_sim no)
@@
 		)
 	)
+	(text "NEXT:\n+Finish calculating current/power of LDO\n+Choose bridge rectifier+ transformer following from this"
+		(exclude_from_sim no)
+		(at -111.506 59.69 0)
+		(effects
+			(font
+				(size 1.27 1.27)
+				(color 255 5 19 1)
+			)
+		)
+	)
 	(text "FAN-\n"
 		(exclude_from_sim no)
@@
 		)
 	)
+	(text "Power of the PSU rail:\n"
+		(exclude_from_sim no)
+		(at 446.024 120.142 0)
+		(effects
+			(font
+				(size 1.27 1.27)
+				(thickness 0.254)
+				(bold yes)
+			)
+		)
+	)
 	(text "1-Change components: Packaging, from Git library+ Standard components+ IMPORTANT TO TRY TO REUSE IF IT WORKS what I already have\n	1.1- Connectors need to select considering clearance-Creepage: I have six connectors\n		* 220V AC INPUT- For 15/-15V trafo\n		* 30V AC INPUT - From external trafo and directly to rectifier\n		* Output of the PSU- +- Terminals (Can be +30V/5A)\n		* Fan Supply OUTPUT- Try to test at 15V \n		* V_ref-I_ref INPUT (With 5V OUTPUT)\n		* V_out and I_out measurements OUTPUT to PSU_Monitoring\n2- Power supplies: +-15V, 12V (needed), and 5V (step by step)\n	2.1- Be carefull on all the packaging\n3- Need to check manufacturing rules\n	3.1- Check testpoint and vias minimum size"
 		(exclude_from_sim no)
@@
 		)
 	)
+	(text "Write down properties of the trnasformer here"
+		(exclude_from_sim no)
+		(at 14.478 77.978 0)
+		(effects
+			(font
+				(size 1.27 1.27)
+				(color 255 29 56 1)
+			)
+		)
+	)
 	(text "GO BACKWARDS: START FROM LDO's TO BRIDGE RECTIFIER CURRENT, AND THEN TRAFO POWER AND CONNECTOR"
 		(exclude_from_sim no)
@@
 		)
 	)
+	(text "+30V*5A=150W"
+		(exclude_from_sim no)
+		(at 444.754 123.698 0)
+		(effects
+			(font
+				(size 1.27 1.27)
+				(thickness 0.1588)
+			)
+		)
+	)
 	(text "holes\n"
 		(exclude_from_sim no)
@@
 		)
 	)
+	(text "P_out=150W\nWith heat sink:15A \nWIthout heatsin:3.2A!! "
+		(exclude_from_sim no)
+		(at 98.552 69.088 0)
+		(effects
+			(font
+				(size 1.27 1.27)
+			)
+		)
+	)
 	(text "* Fan: Need to calculate @home. For the moment lets say 1A\n* Voltage presence indicator: 20mA\n* Mosfet Gate driver: Imax-=0.5A\n	> When MOSFET fully closed (Current dissipated in 20Ω): 6V/20Ω=0.3A\n	> When MOSFET fully opened (Current dissipated in 10Ω+ Diode voltage drop): (6V-1V)/10Ω=0.5A\n* LDO 5V: P_int_LDO_5V+ P_out_5V= (V_in-V_out)*I_out + V_in*Iq (Quiescent current)= 7*1A+12V*3.2mA= 7.0384W+1.35W\n* P_out_12V= [12V * (1+20e-3+0.5)]+8.3884= 26.6284W\n"
 		(exclude_from_sim no)
@@
 		)
 	)
+	(text "Regulable Lab Power Supply Unit (PSU): 30V/5A"
+		(exclude_from_sim no)
+		(at 208.28 1.27 0)
+		(effects
+			(font
+				(size 2.54 2.54)
+				(thickness 0.3556)
+				(bold yes)
+			)
+		)
+	)
 	(text "ALREADY DONE\n"
 		(exclude_from_sim no)
@@
 	)
 	(symbol
+		(lib_id "m_BridgeRectifier:KBJB1506_T0_00301")
+		(at 64.77 68.58 0)
+		(unit 1)
+		(exclude_from_sim no)
+		(in_bom yes)
+		(on_board yes)
+		(dnp no)
+		(property "Reference" "BR5"
+			(at 73.914 63.5 0)
+			(effects
+				(font
+					(size 1.27 1.27)
+				)
+				(justify left top)
+			)
+		)
+		(property "Value" "KBJB1506_T0_00301"
+			(at 66.294 79.502 0)
+			(effects
+				(font
+					(size 1.27 1.27)
+				)
+				(justify left top)
+			)
+		)
+		(property "Footprint" "m_BridgeRectifier:KBJB1506_T0_00301"
+			(at 83.82 163.5 0)
+			(effects
+				(font
+					(size 1.27 1.27)
+				)
+				(justify left top)
+				(hide yes)
+			)
+		)
+		(property "Datasheet" "https://www.panjit.com.tw/upload/datasheet/KBJB1506.pdf?fbclid=IwZXh0bgNhZW0CMTEAAR4OZ1Fo33rf7qdomQ3aAz3Y4ejb0yMDtPrprgTzLzOFng4Hasfgi1CcWfysow_aem_eSJzpmnXgLvNSM2pT6vx4g"
+			(at 83.82 263.5 0)
+			(effects
+				(font
+					(size 1.27 1.27)
+				)
+				(justify left top)
+				(hide yes)
+			)
+		)
+		(property "Description" "Bridge Rectifiers Glass Passivated Low Profile Bridge Rectifier 600V, 15A"
+			(at 64.77 68.58 0)
+			(effects
+				(font
+					(size 1.27 1.27)
+				)
+				(hide yes)
+			)
+		)
+		(property "Height" "12"
+			(at 83.82 463.5 0)
+			(effects
+				(font
+					(size 1.27 1.27)
+				)
+				(justify left top)
+				(hide yes)
+			)
+		)
+		(property "Mouser Part Number" "241-KBJB1506T00301"
+			(at 83.82 563.5 0)
+			(effects
+				(font
+					(size 1.27 1.27)
+				)
+				(justify left top)
+				(hide yes)
+			)
+		)
+		(property "Mouser Price/Stock" "https://www.mouser.co.uk/ProductDetail/Panjit/KBJB1506_T0_00301?qs=VVKQmw408U971kSeRhdwTA%3D%3D"
+			(at 83.82 663.5 0)
+			(effects
+				(font
+					(size 1.27 1.27)
+				)
+				(justify left top)
+				(hide yes)
+			)
+		)
+		(property "Manufacturer_Name" "PANJIT"
+			(at 83.82 763.5 0)
+			(effects
+				(font
+					(size 1.27 1.27)
+				)
+				(justify left top)
+				(hide yes)
+			)
+		)
+		(property "Manufacturer_Part_Number" "KBJB1506_T0_00301"
+			(at 83.82 863.5 0)
+			(effects
+				(font
+					(size 1.27 1.27)
+				)
+				(justify left top)
+				(hide yes)
+			)
+		)
+		(pin "1"
+		)
+		(pin "4"
+		)
+		(pin "3"
+		)
+		(pin "2"
+		)
+		(instances
+			(project ""
+				(path "/47083ad7-9fa0-4f9a-906f-7d13aa6ff8f4"
+					(reference "BR5")
+					(unit 1)
+				)
+			)
+		)
+	)
+	(symbol
 		(lib_id "power:+15V")
 		(at 67.31 166.37 0)
@@
 					(unit 1)
 				)
-			)
-		)
-	)
-	(symbol
-		(lib_id "KBJB1506_T0_00301:KBJB1506_T0_00301")
-		(at 64.77 68.58 0)
-		(unit 1)
-		(exclude_from_sim no)
-		(in_bom yes)
-		(on_board yes)
-		(dnp no)
-		(property "Reference" "BR4"
-			(at 73.406 64.516 0)
-			(effects
-				(font
-					(size 1.27 1.27)
-				)
-				(justify left)
-			)
-		)
-		(property "Value" "KBJB1506_T0_00301"
-			(at 64.008 80.264 0)
-			(effects
-				(font
-					(size 1.27 1.27)
-				)
-				(justify left)
-			)
-		)
-		(property "Footprint" "USER_BRIDGE_RECTIFIER_2:KBJB1506_T0_00301"
-			(at 83.82 163.5 0)
-			(effects
-				(font
-					(size 1.27 1.27)
-				)
-				(justify left top)
-				(hide yes)
-			)
-		)
-		(property "Datasheet" "https://www.panjit.com.tw/upload/datasheet/KBJB1506.pdf?fbclid=IwZXh0bgNhZW0CMTEAAR4OZ1Fo33rf7qdomQ3aAz3Y4ejb0yMDtPrprgTzLzOFng4Hasfgi1CcWfysow_aem_eSJzpmnXgLvNSM2pT6vx4g"
-			(at 83.82 263.5 0)
-			(effects
-				(font
-					(size 1.27 1.27)
-				)
-				(justify left top)
-				(hide yes)
-			)
-		)
-		(property "Description" "Bridge Rectifiers Glass Passivated Low Profile Bridge Rectifier 600V, 15A"
-			(at 64.77 68.58 0)
-			(effects
-				(font
-					(size 1.27 1.27)
-				)
-				(hide yes)
-			)
-		)
-		(property "Height" "12"
-			(at 83.82 463.5 0)
-			(effects
-				(font
-					(size 1.27 1.27)
-				)
-				(justify left top)
-				(hide yes)
-			)
-		)
-		(property "Mouser Part Number" "241-KBJB1506T00301"
-			(at 83.82 563.5 0)
-			(effects
-				(font
-					(size 1.27 1.27)
-				)
-				(justify left top)
-				(hide yes)
-			)
-		)
-		(property "Mouser Price/Stock" "https://www.mouser.co.uk/ProductDetail/Panjit/KBJB1506_T0_00301?qs=VVKQmw408U971kSeRhdwTA%3D%3D"
-			(at 83.82 663.5 0)
-			(effects
-				(font
-					(size 1.27 1.27)
-				)
-				(justify left top)
-				(hide yes)
-			)
-		)
-		(property "Manufacturer_Name" "PANJIT"
-			(at 83.82 763.5 0)
-			(effects
-				(font
-					(size 1.27 1.27)
-				)
-				(justify left top)
-				(hide yes)
-			)
-		)
-		(property "Manufacturer_Part_Number" "KBJB1506_T0_00301"
-			(at 83.82 863.5 0)
-			(effects
-				(font
-					(size 1.27 1.27)
-				)
-				(justify left top)
-				(hide yes)
-			)
-		)
-		(pin "3"
-		)
-		(pin "1"
-		)
-		(pin "2"
-		)
-		(pin "4"
-		)
-		(instances
-			(project "PowerSupply30V5A"
-				(path "/47083ad7-9fa0-4f9a-906f-7d13aa6ff8f4"
-					(reference "BR4")
-					(unit 1)
-				)
