File: PowerSupply30V5A.kicad_sch (KiCad schematic)
At the start: 159 parts, among them IC1 MC7805BDTRKG, IC10 LF247DT, IC2 MC7815BDTRKG, IC3 MC7915BD2TR4G, IC4 MC7815BDTRKG, IC5 MC7812BDTRKG, IC6 MC7805BDTRKG, IC7 MC7915BD2TR4G, IC8 LF247DT, IC9 MC7812BDTRKG, J1 1017503, J10 1755752, J11 1017503, J12 ${FAMILY}, J2 1017503, J3 76825-0004, J4 39300020, J5 76825-0004, J6 1017503, J7 ${FAMILY}, J8 ${FAMILY}, J9 1755752, Q1 IRFP460, Q3 IRFP460, T1 AVB2.3_2_15, U1 ADA4062-2ARMZ, U2 ADA4062-2ARMZ, U3 ADA4062-2ARMZ

Commit message: small comment:
Connections:
- net at R37. (2): now also IC8.2 (-), R36. (2); no longer R38. (2)
- net at R49. (2): now also IC8.6 (-), R48. (2); no longer R50. (2)
- new net: R37. (2), R38. (2)
- new net: R49. (2), R50. (2)
- new net: C36. (2), IC8.13 (-), R55. (2), R56. (2)
- new net: IC8.10 (+), R39. (2), R40. (2)
- new net: C34. (2), IC8.12 (+), R53. (2), R54. (2)
- new net: IC8.3 (+), R30. (2), R44. (2)
- new net: C32. (2), IC8.5 (+), R47. (2), R51. (2)
- new net: C33. (2), IC8.9 (-), R41. (2), R42. (2)
Other:
- note added: "learn to derive pk, rms , avg"
Changed lines of the file:
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@@
+		)
+	)
+	(text "learn to derive pk, rms , avg"
+		(exclude_from_sim no)
+		(at -121.92 66.548 0)
+		(effects
+			(font
+				(size 1.27 1.27)
+				(thickness 0.254)
+				(bold yes)
+			)
 		)
 	)

Commit message: Measured fan current
Connections:
- net at R37. (2): now also IC8.2 (-), R36. (2); no longer R38. (2)
- net at R49. (2): now also IC8.6 (-), R48. (2); no longer R50. (2)
- new net: R37. (2), R38. (2)
- new net: R49. (2), R50. (2)
- new net: C36. (2), IC8.13 (-), R55. (2), R56. (2)
- new net: IC8.10 (+), R39. (2), R40. (2)
- new net: C34. (2), IC8.12 (+), R53. (2), R54. (2)
- new net: IC8.3 (+), R30. (2), R44. (2)
- new net: C32. (2), IC8.5 (+), R47. (2), R51. (2)
- new net: C33. (2), IC8.9 (-), R41. (2), R42. (2)
Other:
- note added: "* Fan: 0.28A * Voltage presence indicator: 20mA * Mosfet Gate driver: Imax-=0.5A > When MOSFET fully closed (Current dissipated in 20Ω): 6V/20Ω=0.3A > When MOSFET fully opened (Current dissipated in 10Ω+ Diode voltage drop): (6V-1V)/10Ω=0.5A * LDO 5V: P_int_LDO_5V+ P_out_5V= (V_in-V_out)*I_out + V_in*Iq (Quiescent current)= 7*1A+12V*3.2mA= 7.0384W+1.35W * P_out_12V= [12V * (0.28+20e-3+0.5)]+8.388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"
- note added: "* Voltage presence indicator: 20mA * Quad op-amp buffer: 680mW Pmax when output @+15V * Quad op-amp voltage and current PI:680mW Pmax when output @+15V * LDO 12V: P_int_LDO_12V+P_out_12V= (V_in-V_out)*I_out + V_in*Iq (Quiescent current)= 3V*1A+18V*3.5mA= 3.063W+18W * P_tot_15V:21,0514W+15*20e-3+(2*680e-3)=22,7114"
- note added: "+12V: (18W)"
- note added: "+15V: (23W)"
- note added: "+30V*5A=150W Power of first bridge rectifier"
- note added: "+5V: (1.5W)"
- note added: "-15V: (2W)"
- note added: "I_out_15V=1.54A"
- note added: "NEXT: +Need to change two LDO: Higher power +Choose bridge rectifier+ transformer following from this"
- note added: "Total power of second bridge rectifier: P_tot=1.5+18+23+20=44.5==45W"
- note removed: "* Fan: Need to calculate @home. For the moment lets say 1A * Voltage presence indicator: 20mA * Mosfet Gate driver: Imax-=0.5A > When MOSFET fully closed (Current dissipated in 20Ω): 6V/20Ω=0.3A > When MOSFET fully opened (Current dissipated in 10Ω+ Diode voltage drop): (6V-1V)/10Ω=0.5A * LDO 5V: P_int_LDO_5V+ P_out_5V= (V_in-V_out)*I_out + V_in*Iq (Quiescent current)= 7*1A+12V*3.2mA= 7.0384W+1.3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"
- note removed: "* Voltage presence indicator: 20mA * Quad op-amp buffer: 680mW Pmax when output @+15V * Quad op-amp voltage and current PI:680mW Pmax when output @+15V * LDO 12V: P_int_LDO_12V+P_out_12V= (V_in-V_out)*I_out + V_in*Iq (Quiescent current)= 3V*1A+18V*3.5mA= 3.063W * P_tot_15V"
- note removed: "+12V: (20.27W)"
- note removed: "+15V: (xx W)"
- note removed: "+30V*5A=150W"
- note removed: "+5V: (1.35W)"
- note removed: "-15V: (xx W)"
- note removed: "Claro, el opamp es 1A solo, asique tengo que medir esto. Si es 1A, tengo que cambiar LDO Aqui estoy dando 2A en el op-amp! no funciona"
- note removed: "I_out_15V=xxA"
- note removed: "NEXT: +Finish calculating current/power of LDO +Choose bridge rectifier+ transformer following from this"
- note removed: "Y aqui cambiar P_out_12V una vez haya medido"
Changed lines of the file:
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@@
-		)
-	)
-	(text "Y aqui cambiar P_out_12V una vez haya medido"
-		(exclude_from_sim no)
-		(at 588.518 90.424 0)
-		(effects
-			(font
-				(size 1.27 1.27)
-				(color 255 51 72 1)
-			)
 		)
 	)
@@
 		)
 	)
-	(text "+15V: (xx W)"
+	(text "+15V: (23W)"
 		(exclude_from_sim no)
 		(at 442.722 81.534 0)
@@
 		)
 	)
-	(text "+12V: (20.27W)"
+	(text "+12V: (18W)"
 		(exclude_from_sim no)
 		(at 443.484 60.96 0)
@@
 		)
 	)
-	(text "* Voltage presence indicator: 20mA\n* Quad op-amp buffer: 680mW Pmax when output @+15V\n* Quad op-amp voltage and current PI:680mW Pmax when output @+15V\n* LDO 12V: P_int_LDO_12V+P_out_12V= (V_in-V_out)*I_out + V_in*Iq (Quiescent current)= 3V*1A+18V*3.5mA= 3.063W\n* P_tot_15V"
+	(text "* Voltage presence indicator: 20mA\n* Quad op-amp buffer: 680mW Pmax when output @+15V\n* Quad op-amp voltage and current PI:680mW Pmax when output @+15V\n* LDO 12V: P_int_LDO_12V+P_out_12V= (V_in-V_out)*I_out + V_in*Iq (Quiescent current)= 3V*1A+18V*3.5mA= 3.063W+18W\n* P_tot_15V:21,0514W+15*20e-3+(2*680e-3)=22,7114"
 		(exclude_from_sim no)
 		(at 436.88 88.646 0)
@@
 		)
 	)
-	(text "NEXT:\n+Finish calculating current/power of LDO\n+Choose bridge rectifier+ transformer following from this"
+	(text "NEXT:\n+Need to change two LDO: Higher power\n+Choose bridge rectifier+ transformer following from this"
 		(exclude_from_sim no)
 		(at -111.506 59.69 0)
@@
 		)
 	)
-	(text "Claro, el opamp es 1A solo, asique tengo que medir esto. Si es 1A, tengo que cambiar LDO\nAqui estoy dando 2A en el op-amp! no funciona"
-		(exclude_from_sim no)
-		(at 546.862 77.724 0)
-		(effects
-			(font
-				(size 1.27 1.27)
-				(color 255 1 15 1)
-			)
-		)
-	)
 	(text "P_max_operation=1.25W(50mOhms*(5A)^2)\n"
 		(exclude_from_sim no)
@@
 		)
 	)
-	(text "I_out_15V=xxA"
-		(exclude_from_sim no)
-		(at 446.024 95.504 0)
+	(text "I_out_15V=1.54A"
+		(exclude_from_sim no)
+		(at 447.802 94.996 0)
 		(effects
 			(font
@@
 		)
 	)
+	(text "Total power of second bridge rectifier: \nP_tot=1.5+18+23+20=44.5==45W"
+		(exclude_from_sim no)
+		(at 437.642 120.396 0)
+		(effects
+			(font
+				(size 1.27 1.27)
+			)
+			(justify left)
+		)
+	)
 	(text "DUDAS:\nAnalogue 0 connected to GND? (ok)\n"
 		(exclude_from_sim no)
@@
 	(text "Power of the PSU rail:\n"
 		(exclude_from_sim no)
-		(at 446.024 120.142 0)
+		(at 448.564 126.492 0)
 		(effects
 			(font
@@
 		)
 	)
-	(text "+30V*5A=150W"
-		(exclude_from_sim no)
-		(at 444.754 123.698 0)
+	(text "+30V*5A=150W\nPower of first bridge rectifier"
+		(exclude_from_sim no)
+		(at 437.388 130.81 0)
 		(effects
 			(font
@@
 				(thickness 0.1588)
 			)
+			(justify left)
 		)
 	)
@@
 		)
 	)
-	(text "-15V: (xx W)"
-		(exclude_from_sim no)
-		(at 443.992 100.076 0)
+	(text "-15V: (2W)"
+		(exclude_from_sim no)
+		(at 442.468 102.362 0)
 		(effects
 			(font
@@
 		)
 	)
-	(text "* Fan: Need to calculate @home. For the moment lets say 1A\n* Voltage presence indicator: 20mA\n* Mosfet Gate driver: Imax-=0.5A\n	> When MOSFET fully closed (Current dissipated in 20Ω): 6V/20Ω=0.3A\n	> When MOSFET fully opened (Current dissipated in 10Ω+ Diode voltage drop): (6V-1V)/10Ω=0.5A\n* LDO 5V: P_int_LDO_5V+ P_out_5V= (V_in-V_out)*I_out + V_in*Iq (Quiescent current)= 7*1A+12V*3.2mA= 7.0384W+1.35W\n* P_out_12V= [12V * (1+20e-3+0.5)]+8.3884= 26.6284W\n"
+	(text "* Fan: 0.28A\n* Voltage presence indicator: 20mA\n* Mosfet Gate driver: Imax-=0.5A\n	> When MOSFET fully closed (Current dissipated in 20Ω): 6V/20Ω=0.3A\n	> When MOSFET fully opened (Current dissipated in 10Ω+ Diode voltage drop): (6V-1V)/10Ω=0.5A\n* LDO 5V: P_int_LDO_5V+ P_out_5V= (V_in-V_out)*I_out + V_in*Iq (Quiescent current)= 7*1A+12V*3.2mA= 7.0384W+1.35W\n* P_out_12V= [12V * (0.28+20e-3+0.5)]+8.3884= 18W\n"
 		(exclude_from_sim no)
 		(at 438.15 70.104 0)
@@
 		)
 	)
-	(text "+5V: (1.35W)"
+	(text "+5V: (1.5W)"
 		(exclude_from_sim no)
 		(at 441.96 42.926 0)

Commit message: Included new LDO
Parts:
- added IC11: BDJ2FD0WHFP-TR, m_LDO:BDJ2FD0WHFPTR, symbol m_LDO:BDJ2FD0WHFP-TR
- added IC12: BDJ5FD0WHFP-TR, m_LDO:BDJ5FD0WHFPTR, symbol m_LDO:BDJ5FD0WHFP-TR
Connections:
- net at R37. (2): now also IC8.2 (-), R36. (2); no longer R38. (2)
- net at R49. (2): now also IC8.6 (-), R48. (2); no longer R50. (2)
- new net: R37. (2), R38. (2)
- new net: R49. (2), R50. (2)
- new net: C36. (2), IC8.13 (-), R55. (2), R56. (2)
- new net: IC8.10 (+), R39. (2), R40. (2)
- new net: C34. (2), IC8.12 (+), R53. (2), R54. (2)
- new net: IC8.3 (+), R30. (2), R44. (2)
- new net: C32. (2), IC8.5 (+), R47. (2), R51. (2)
- new net: C33. (2), IC8.9 (-), R41. (2), R42. (2)
Other:
- note added: "* Fan: 0.28A * Voltage presence indicator: 20mA * Mosfet Gate driver: Imax-=0.5A > When MOSFET fully closed (Current dissipated in 20Ω): 6V/20Ω=0.3A > When MOSFET fully opened (Current dissipated in 10Ω+ Diode voltage drop): (6V-1V)/10Ω=0.5A * LDO 5V: P_int_LDO_5V+ P_out_5V= V_in*Iq (Quiescent current)+ (V_in-V_out)*I_out= 12V*3.2mA+ 7*1A= 7.0384W+1.35W * P_out_12V= [12V * (0.28+20e-3+0.5)]+8.388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"
- note added: "* Voltage presence indicator: 20mA * Quad op-amp buffer: 680mW Pmax when output @+15V * Quad op-amp voltage and current PI:680mW Pmax when output @+15V * LDO 12V: P_int_LDO_12V+P_out_12V= V_in*Iq (Quiescent current)+(V_in-V_out)*I_out= 15V*0.5mA+3V*1.5A= 4.5W+18W * P_tot_15V:21,0514W+15*20e-3+(2*680e-3)=22,5"
- note added: "I_out_12V=1.5A"
- note added: "I_out_15V=1.5A"
- note added: "NEXT: +Need to change two LDO: Higher power, HIGHER CURRENT +Choose bridge rectifier+ transformer following from this"
- note added: "The voltage regulation was not okey because too much power, it was turning down the LDO´s"
- note added: "Total power of second bridge rectifier: P_tot=1.5+18+23+2=44.5==45W"
- note removed: "* Fan: 0.28A * Voltage presence indicator: 20mA * Mosfet Gate driver: Imax-=0.5A > When MOSFET fully closed (Current dissipated in 20Ω): 6V/20Ω=0.3A > When MOSFET fully opened (Current dissipated in 10Ω+ Diode voltage drop): (6V-1V)/10Ω=0.5A * LDO 5V: P_int_LDO_5V+ P_out_5V= (V_in-V_out)*I_out + V_in*Iq (Quiescent current)= 7*1A+12V*3.2mA= 7.0384W+1.35W * P_out_12V= [12V * (0.28+20e-3+0.5)]+8.388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"
- note removed: "* Voltage presence indicator: 20mA * Quad op-amp buffer: 680mW Pmax when output @+15V * Quad op-amp voltage and current PI:680mW Pmax when output @+15V * LDO 12V: P_int_LDO_12V+P_out_12V= (V_in-V_out)*I_out + V_in*Iq (Quiescent current)= 3V*1A+18V*3.5mA= 3.063W+18W * P_tot_15V:21,0514W+15*20e-3+(2*680e-3)=22,7114"
- note removed: "I_out_12V=2A"
- note removed: "I_out_15V=1.54A"
- note removed: "NEXT: +Need to change two LDO: Higher power +Choose bridge rectifier+ transformer following from this"
- note removed: "Total power of second bridge rectifier: P_tot=1.5+18+23+20=44.5==45W"

Commit message: Changed LDO, now need to change trafo and bridge rectifier, all the ratings
Parts:
- removed C20: 330nF_25V, m_Capacitor_ceramic_SMD:CAPC2012X94N, symbol m_Capacitor_ceramic_SMD:0805_330nF_25V_10%
- removed C37: 1μF_25V, m_Capacitor_ceramic_SMD:CAPC2012X94N, symbol m_Capacitor_ceramic_SMD:0805_1μF_25V_20%
- removed IC2: MC7815BDTRKG, m_LDO:NVD5117PLT4GVF01, symbol m_LDO:MC7815BDTRKG
- removed TP12: TestPoint, Connector_Pin:Pin_D0.7mm_L6.5mm_W1.8mm_FlatFork, symbol Connector:TestPoint
- added C20, C39: 1μF_25V, m_Capacitor_ceramic_SMD:CAPC2012X94N, symbol m_Capacitor_ceramic_SMD:0805_1μF_25V_20%
- added C37, C40: 4.7uF_25V, m_Capacitor_ceramic_SMD:CAPC2012X94N, symbol m_Capacitor_ceramic_SMD:0805_4.7uF_25V_20%
Connections:
- net +12V: now also IC11.4 (VO), C40. (2)
- net +15V: now also IC11.1 (CTL), IC11.2 (VCC), IC12.4 (VO), C37. (2), C39. (2)
- net GND: now also IC11.3 (GND), IC11.5 (N.C._), IC11.6 (FIN), IC12.3 (GND), IC12.5 (N.C.), IC12.6 (FIN), C20. (2), C37. (2), C39. (2), C40. (2)
- net at R37. (2): now also IC8.2 (-), R36. (2); no longer R38. (2)
- net at R49. (2): now also IC8.6 (-), R48. (2); no longer R50. (2)
- net at C17.1: now also IC12.1 (CTL), IC12.2 (VCC), C20. (2)
- new net: R37. (2), R38. (2)
- new net: R49. (2), R50. (2)
- new net: C36. (2), IC8.13 (-), R55. (2), R56. (2)
- new net: IC8.10 (+), R39. (2), R40. (2)
- new net: C34. (2), IC8.12 (+), R53. (2), R54. (2)
- new net: IC8.3 (+), R30. (2), R44. (2)
- new net: C32. (2), IC8.5 (+), R47. (2), R51. (2)
- new net: C33. (2), IC8.9 (-), R41. (2), R42. (2)
Other:
- note added: "DEBERÍA DE TENER SIMETRICO 15-15V ? De todos modos voy a tener diferentes corrientes. Asi que no veo porque debería de afectar diferente componente. Por ahora dejar así"
- note added: "Follow datasheet for this"
- note added: "I_out(max): 2A"
- note added: "LDO Dropout voltage: 0.4V So for 15V I need 15.6Vmin in the output"
- note added: "LDO dropout voltage: 0.4V So for 12v I need 12.6Vmin"
- note added: "NEXT: +Choose bridge rectifier+ transformer following change of LDO"
- note added: "Total power of second bridge rectifier: P_tot=1.5+18+23+2=44.5==45W REMEMBER THAT TO SUPPLY ALL THE LDO´S, i might need more than 30V, probably +36V would be approapiate"
- note removed: "LDO Dropout voltage: 2V So for 15V I need 18Vmin in the output"
- note removed: "NEXT: +Need to change two LDO: Higher power, HIGHER CURRENT +Choose bridge rectifier+ transformer following from this"
- note removed: "Total power of second bridge rectifier: P_tot=1.5+18+23+2=44.5==45W"
- moved on the sheet: C23, C24, IC11, IC9, TP14
